Commit message: a

File: simulation/lendoc/map20/map20lendoc/urdf/map20.urdf (robot description, URDF)
Before this commit: robot map25xuongdoc, 1 links, 0 joints
Links:
- link base_link: geometry collision mesh filename=package://map20lendoc/meshes/base_link.STL; visual mesh filename=package://map20lendoc/meshes/base_link.STL

File: simulation/lendoc/map25/map25lendoc/urdf/map25.urdf (robot description, URDF)
Before this commit: robot map25xuongdoc, 1 links, 0 joints
Links:
- link base_link: mass 41.50417784345 -> 40.0170338495876; geometry collision mesh filename=package://map25lendoc/meshes/base_link.STL; visual mesh filename=package://map25lendoc/meshes/base_link.STL

File: simulation/lendoc/map30/map30lendoc/urdf/map30.urdf (robot description, URDF)
Before this commit: robot map25xuongdoc, 1 links, 0 joints
Links:
- link base_link: mass 41.50417784345 -> 39.0165244785435; geometry collision mesh filename=package://map30lendoc/meshes/base_link.STL; visual mesh filename=package://map30lendoc/meshes/base_link.STL
